File: Hardware/SparkFun_Qwiic_Buzzer.sch (EAGLE design)
At the start: 45 parts, among them J2 QWIIC_RA, J3 QWIIC_RA, Q3 200mA/40V, U4 ATTINY84-ARDUINO

Commit message: final review tweaks - no copper changes
-re-order position of 0.1uF and 10uF Caps
-re-order vol resistors
-redo measures so they are better
-added QWIIC logo to sch
Parts:
- added LOGO5: QWIIC_LOGO_4MM, SparkFun-Aesthetics:QWIIC_LOGO_4MM
- R15: value 100 -> 2.2k; device SparkFun-Resistors:100OHM-0402-TIGHT-1/16W-1% -> SparkFun-Resistors:2.2KOHM-0402T-1/16W-1%
- R17: value 2.2k -> 100; device SparkFun-Resistors:2.2KOHM-0402T-1/16W-1% -> SparkFun-Resistors:100OHM-0402-TIGHT-1/16W-1%
Other:
- note added: "ATTINY VCC: 1.8-5.5V (Typically 3.3V from QWIIC) Buzzer: 2.5-4.5V"
- note removed: "VCC: 1.8-5.5V (Typically 3.3V from QWIIC)"
- moved on the sheet: C1, C2
Changed lines of the file:
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@@
 <part name="R12" library="SparkFun-Resistors" deviceset="330OHM" device="-0402T-1/16W-5%" value="330"/>
 <part name="R13" library="SparkFun-Resistors" deviceset="330OHM" device="-0402T-1/16W-5%" value="330"/>
-<part name="R17" library="SparkFun-Resistors" deviceset="2.2KOHM" device="-0402T-1/16W-1%" value="2.2k"/>
+<part name="R17" library="SparkFun-Resistors" deviceset="100OHM" device="-0402-TIGHT-1/16W-1%" value="100"/>
 <part name="R14" library="SparkFun-Resistors" deviceset="330OHM" device="-0402T-1/16W-5%" value="330"/>
-<part name="R15" library="SparkFun-Resistors" deviceset="100OHM" device="-0402-TIGHT-1/16W-1%" value="100"/>
+<part name="R15" library="SparkFun-Resistors" deviceset="2.2KOHM" device="-0402T-1/16W-1%" value="2.2k"/>
 <part name="GND1" library="SparkFun-PowerSymbols" deviceset="GND" device=""/>
 <part name="H3" library="SparkFun-Hardware" deviceset="STAND-OFF" device=""/>
@@
 <part name="JP1" library="SparkFun-Jumpers" deviceset="JUMPER-SMT_2_NC_TRACE" device="_SILK" package3d_urn="urn:adsk.eagle:package:39281/1" value=""/>
 <part name="J6" library="SparkFun-Connectors" deviceset="CONN_03" device="1X03_NO_SILK"/>
+<part name="LOGO5" library="SparkFun-Aesthetics" deviceset="QWIIC_LOGO" device="_4MM"/>
 </parts>
 <sheets>
@@
 <wire x1="147.32" y1="99.06" x2="0" y2="99.06" width="0.1524" layer="97" style="longdash"/>
 <text x="2.54" y="93.98" size="2.54" layer="94" font="vector">Buzzer</text>
-<text x="2.54" y="177.8" size="1.27" layer="97" font="vector">VCC: 1.8-5.5V (Typically 3.3V from QWIIC)</text>
+<text x="2.54" y="175.26" size="1.27" layer="97" font="vector">ATTINY VCC: 1.8-5.5V (Typically 3.3V from QWIIC)
+Buzzer: 2.5-4.5V</text>
 <text x="148.844" y="6.096" size="2.54" layer="94" font="vector">Based on designed by:</text>
 <text x="166.116" y="11.176" size="2.54" layer="94" font="vector">Pete Lewis</text>
@@
 <attribute name="NAME" x="193.04" y="101.092" size="1.778" layer="95" font="vector" rot="R180"/>
 </instance>
-<instance part="GND7" gate="1" x="33.02" y="139.7" smashed="yes">
-<attribute name="VALUE" x="30.48" y="137.16" size="1.778" layer="96" font="vector"/>
-</instance>
-<instance part="C2" gate="G$1" x="33.02" y="147.32" smashed="yes">
-<attribute name="NAME" x="34.544" y="150.241" size="1.778" layer="95" font="vector"/>
-<attribute name="VALUE" x="34.544" y="145.161" size="1.778" layer="96" font="vector"/>
+<instance part="GND7" gate="1" x="43.18" y="139.7" smashed="yes">
+<attribute name="VALUE" x="40.64" y="137.16" size="1.778" layer="96" font="vector"/>
+</instance>
+<instance part="C2" gate="G$1" x="43.18" y="147.32" smashed="yes">
+<attribute name="NAME" x="44.704" y="150.241" size="1.778" layer="95" font="vector"/>
+<attribute name="VALUE" x="44.704" y="145.161" size="1.778" layer="96" font="vector"/>
 </instance>
 <instance part="R2" gate="G$1" x="119.38" y="147.32" smashed="yes" rot="R90">
@@
 <attribute name="VALUE" x="45.72" y="66.548" size="1.27" layer="96" font="vector" rot="MR0" align="top-left"/>
 </instance>
-<instance part="C1" gate="G$1" x="43.18" y="147.32" smashed="yes">
-<attribute name="NAME" x="44.704" y="150.241" size="1.778" layer="95" font="vector"/>
-<attribute name="VALUE" x="44.704" y="145.161" size="1.778" layer="96" font="vector"/>
-</instance>
-<instance part="GND3" gate="1" x="43.18" y="139.7" smashed="yes">
-<attribute name="VALUE" x="40.64" y="137.16" size="1.778" layer="96" font="vector"/>
+<instance part="C1" gate="G$1" x="33.02" y="147.32" smashed="yes">
+<attribute name="NAME" x="34.544" y="150.241" size="1.778" layer="95" font="vector"/>
+<attribute name="VALUE" x="34.544" y="145.161" size="1.778" layer="96" font="vector"/>
+</instance>
+<instance part="GND3" gate="1" x="33.02" y="139.7" smashed="yes">
+<attribute name="VALUE" x="30.48" y="137.16" size="1.778" layer="96" font="vector"/>
 </instance>
 <instance part="JP1" gate="G$1" x="106.68" y="48.26" smashed="yes" rot="R180">
@@
 <attribute name="NAME" x="220.98" y="101.092" size="1.778" layer="95" font="vector" rot="R180"/>
 </instance>
+<instance part="LOGO5" gate="G$1" x="236.22" y="58.42" smashed="yes"/>
 </instances>
 <busses>
@@
 </segment>
 <segment>
-<wire x1="33.02" y1="144.78" x2="33.02" y2="142.24" width="0.1524" layer="91"/>
+<wire x1="43.18" y1="144.78" x2="43.18" y2="142.24" width="0.1524" layer="91"/>
 <pinref part="GND7" gate="1" pin="GND"/>
 <pinref part="C2" gate="G$1" pin="2"/>
@@
 <segment>
 <pinref part="C1" gate="G$1" pin="2"/>
-<wire x1="43.18" y1="144.78" x2="43.18" y2="142.24" width="0.1524" layer="91"/>
+<wire x1="33.02" y1="144.78" x2="33.02" y2="142.24" width="0.1524" layer="91"/>
 <pinref part="GND3" gate="1" pin="GND"/>
 </segment>
@@
 <pinref part="SUPPLY17" gate="G$1" pin="3.3V"/>
 <pinref part="U4" gate="U1" pin="VCC"/>
-<wire x1="33.02" y1="152.4" x2="33.02" y2="154.94" width="0.1524" layer="91"/>
 <pinref part="C2" gate="G$1" pin="1"/>
 <wire x1="48.26" y1="154.94" x2="43.18" y2="154.94" width="0.1524" layer="91"/>
@@
 <pinref part="C1" gate="G$1" pin="1"/>
 <wire x1="43.18" y1="154.94" x2="33.02" y2="154.94" width="0.1524" layer="91"/>
+<junction x="43.18" y="154.94"/>
 <wire x1="43.18" y1="152.4" x2="43.18" y2="154.94" width="0.1524" layer="91"/>
-<junction x="43.18" y="154.94"/>
-</segment>
-<segment>
+<wire x1="33.02" y1="152.4" x2="33.02" y2="154.94" width="0.1524" layer="91"/>
+</segment>
+<segment>

Commit message: BOM change - control resistors changed to 100 ohm
R7, R5, R17, R12, R9
Parts:
- R12, R13, R5, R7, R8: value 330 -> 100; device SparkFun-Resistors:330OHM-0402T-1/16W-5% -> SparkFun-Resistors:100OHM-0402-TIGHT-1/16W-1%
Changed lines of the file:
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@@
 <part name="LOGO4" library="SparkFun-Aesthetics" deviceset="SFE_LOGO_FLAME" device=".1_INCH"/>
 <part name="LS1" library="SparkFun-Electromechanical" deviceset="BUZZER" device="-SMD" value="BUZZER"/>
-<part name="R5" library="SparkFun-Resistors" deviceset="330OHM" device="-0402T-1/16W-5%" value="330"/>
+<part name="R5" library="SparkFun-Resistors" deviceset="100OHM" device="-0402-TIGHT-1/16W-1%" value="100"/>
 <part name="PWR_LED" library="SparkFun-Jumpers" deviceset="JUMPER-SMT_2_NC_TRACE" device="_SILK" package3d_urn="urn:adsk.eagle:package:39281/1" value="PWR_LED"/>
 <part name="SUPPLY3" library="SparkFun-PowerSymbols" deviceset="3.3V" device=""/>
@@
 <part name="Q2" library="SparkFun-DiscreteSemi" deviceset="TRANS_NPN_DUAL" device="-MBT3904DW1T1"/>
 <part name="Q3" library="SparkFun-DiscreteSemi" deviceset="TRANS_PNP" device="-PMBT3906|MMBT3906L" value="200mA/40V"/>
-<part name="R7" library="SparkFun-Resistors" deviceset="330OHM" device="-0402T-1/16W-5%" value="330"/>
+<part name="R7" library="SparkFun-Resistors" deviceset="100OHM" device="-0402-TIGHT-1/16W-1%" value="100"/>
 <part name="Q1" library="SparkFun-DiscreteSemi" deviceset="TRANS_NPN_DUAL" device="-MBT3904DW1T1"/>
 <part name="SUPPLY4" library="SparkFun-PowerSymbols" deviceset="3.3V" device=""/>
-<part name="R8" library="SparkFun-Resistors" deviceset="330OHM" device="-0402T-1/16W-5%" value="330"/>
-<part name="R12" library="SparkFun-Resistors" deviceset="330OHM" device="-0402T-1/16W-5%" value="330"/>
-<part name="R13" library="SparkFun-Resistors" deviceset="330OHM" device="-0402T-1/16W-5%" value="330"/>
+<part name="R8" library="SparkFun-Resistors" deviceset="100OHM" device="-0402-TIGHT-1/16W-1%" value="100"/>
+<part name="R12" library="SparkFun-Resistors" deviceset="100OHM" device="-0402-TIGHT-1/16W-1%" value="100"/>
+<part name="R13" library="SparkFun-Resistors" deviceset="100OHM" device="-0402-TIGHT-1/16W-1%" value="100"/>
 <part name="R17" library="SparkFun-Resistors" deviceset="100OHM" device="-0402-TIGHT-1/16W-1%" value="100"/>
 <part name="R14" library="SparkFun-Resistors" deviceset="330OHM" device="-0402T-1/16W-5%" value="330"/>
