File: Hardware/Production/SparkFun_Qwiic_Buzzer-Panel.brd (EAGLE design)
At the start: 175 x 117.3 mm, 1470 parts, among them J10 QWIIC_RA, J13 QWIIC_RA, J14 QWIIC_RA, J17 QWIIC_RA, J18 QWIIC_RA, J2 QWIIC_RA, J21 QWIIC_RA, J22 QWIIC_RA, J25 QWIIC_RA, J26 QWIIC_RA, J29 QWIIC_RA, J3 QWIIC_RA, J30 QWIIC_RA, J33 QWIIC_RA, J34 QWIIC_RA, J37 QWIIC_RA, J38 QWIIC_RA, J4 QWIIC_RA, J41 QWIIC_RA, J42 QWIIC_RA, J45 QWIIC_RA, J46 QWIIC_RA, J49 QWIIC_RA, J5 QWIIC_RA, J50 QWIIC_RA, J53 QWIIC_RA, J54 QWIIC_RA, J57 QWIIC_RA, J58 QWIIC_RA, J61 QWIIC_RA, J62 QWIIC_RA, J65 QWIIC_RA, J66 QWIIC_RA, J69 QWIIC_RA, J70 QWIIC_RA, J73 QWIIC_RA, J74 QWIIC_RA, J77 QWIIC_RA, J78 QWIIC_RA, J81 QWIIC_RA, J82 QWIIC_RA, J85 QWIIC_RA, J86 QWIIC_RA, J89 QWIIC_RA, J9 QWIIC_RA, J90 QWIIC_RA, J93 QWIIC_RA, J94 QWIIC_RA, Q11 200mA/40V, Q14 200mA/40V, Q17 200mA/40V, Q20 200mA/40V, Q23 200mA/40V, Q26 200mA/40V, Q29 200mA/40V, Q3 200mA/40V, Q32 200mA/40V, Q35 200mA/40V, Q38 200mA/40V, Q41 200mA/40V, Q44 200mA/40V, Q47 200mA/40V, Q5 200mA/40V, Q50 200mA/40V, Q53 200mA/40V, Q56 200mA/40V, Q59 200mA/40V, Q62 200mA/40V, Q65 200mA/40V, Q68 200mA/40V, Q71 200mA/40V, Q8 200mA/40V, U1 ATTINY84-ARDUINO, U10 ATTINY84-ARDUINO, U11 ATTINY84-ARDUINO, U12 ATTINY84-ARDUINO, U13 ATTINY84-ARDUINO, U14 ATTINY84-ARDUINO, U15 ATTINY84-ARDUINO, U16 ATTINY84-ARDUINO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

Commit message: re-panelized and re-cammed
-all gerbers showed no diffs, so we're good to go.
Parts:
- removed U$409, U$427: (no value), output:##RST##7
- removed U$410, U$428: (no value), output:##TRIG##6
- removed U$411, U$429: (no value), output:USER12
- removed U$412, U$430: (no value), output:#PWR_LED#13
- removed U$413, U$431: (no value), output:#JP1#14
- removed U$414, U$432: (no value), output:BUZZER14
- removed U$415: (no value), output:STAT0
- removed U$416: (no value), output:PWR0
- removed U$418: (no value), SparkFun-Aesthetics:QWIIC_5MM
- removed U$419: (no value), output:BUZZER1
- removed U$420: (no value), output:#I2C#0
- removed U$421, U$422: (no value), output:#GND#0
- removed U$423: (no value), output:#3V3#0
- removed U$424: (no value), output:#SDA#0
- removed U$425: (no value), output:#SCL#0
- removed U$426: (no value), output:#STAT#3
- added LOGO73, LOGO77, LOGO81, LOGO85, LOGO89, LOGO93: OSHW-LOGOMINI, SparkFun-Aesthetics:OSHW-LOGO-MINI
- added LOGO74, LOGO78, LOGO82, LOGO86, LOGO90, LOGO94: SFE_LOGO_FLAME.1_INCH, SparkFun-Aesthetics:SFE_LOGO_FLAME_.1
- added LOGO75, LOGO79, LOGO83, LOGO87, LOGO91, LOGO95: SFE_LOGO_NAME_FLAME.1_INCH, SparkFun-Aesthetics:SFE_LOGO_NAME_FLAME_.1
- added LOGO76, LOGO80, LOGO84, LOGO88, LOGO92: QWIIC_LOGO_4MM, SparkFun-Aesthetics:QWIIC_4MM
- LOGO10, LOGO22, LOGO34, LOGO46, LOGO58, LOGO70: value OSHW-LOGOMINI -> SFE_LOGO_FLAME.1_INCH; device SparkFun-Aesthetics:OSHW-LOGO-MINI -> SparkFun-Aesthetics:SFE_LOGO_FLAME_.1
- LOGO11, LOGO23, LOGO35, LOGO47, LOGO59, LOGO71: value SFE_LOGO_FLAME.1_INCH -> SFE_LOGO_NAME_FLAME.1_INCH; device SparkFun-Aesthetics:SFE_LOGO_FLAME_.1 -> SparkFun-Aesthetics:SFE_LOGO_NAME_FLAME_.1
- LOGO12, LOGO24, LOGO36, LOGO48, LOGO60, LOGO72: value SFE_LOGO_NAME_FLAME.1_INCH -> QWIIC_LOGO_4MM; device SparkFun-Aesthetics:SFE_LOGO_NAME_FLAME_.1 -> SparkFun-Aesthetics:QWIIC_4MM
- LOGO16, LOGO28, LOGO40, LOGO52, LOGO64: value OSHW-LOGOMINI -> QWIIC_LOGO_4MM; device SparkFun-Aesthetics:OSHW-LOGO-MINI -> SparkFun-Aesthetics:QWIIC_4MM
- LOGO17, LOGO29, LOGO41, LOGO53, LOGO65: value SFE_LOGO_FLAME.1_INCH -> OSHW-LOGOMINI; device SparkFun-Aesthetics:SFE_LOGO_FLAME_.1 -> SparkFun-Aesthetics:OSHW-LOGO-MINI
- LOGO18, LOGO30, LOGO42, LOGO54, LOGO6, LOGO66: value SFE_LOGO_NAME_FLAME.1_INCH -> SFE_LOGO_FLAME.1_INCH; device SparkFun-Aesthetics:SFE_LOGO_NAME_FLAME_.1 -> SparkFun-Aesthetics:SFE_LOGO_FLAME_.1
- LOGO19, LOGO31, LOGO43, LOGO55, LOGO67, LOGO7: value OSHW-LOGOMINI -> SFE_LOGO_NAME_FLAME.1_INCH; device SparkFun-Aesthetics:OSHW-LOGO-MINI -> SparkFun-Aesthetics:SFE_LOGO_NAME_FLAME_.1
- LOGO20, LOGO32, LOGO44, LOGO5, LOGO56, LOGO68, LOGO8: value SFE_LOGO_FLAME.1_INCH -> QWIIC_LOGO_4MM; device SparkFun-Aesthetics:SFE_LOGO_FLAME_.1 -> SparkFun-Aesthetics:QWIIC_4MM
- LOGO21, LOGO33, LOGO45, LOGO57, LOGO69, LOGO9: value SFE_LOGO_NAME_FLAME.1_INCH -> OSHW-LOGOMINI; device SparkFun-Aesthetics:SFE_LOGO_NAME_FLAME_.1 -> SparkFun-Aesthetics:OSHW-LOGO-MINI
- LOGO96: value (none) -> QWIIC_LOGO_4MM
- R108, R122, R136, R150, R164, R17, R178, R192, R206, R220, R234, R24, R248, R262, R276, R290, R304, R318, R332, R38, R52, R66, R80, R94: value 2.2k -> 100
- R110, R124, R138, R15, R152, R166, R180, R194, R208, R222, R236, R250, R26, R264, R278, R292, R306, R320, R334, R40, R54, R68, R82, R96: value 100 -> 2.2k
- U$100, U$406: device output:#SDA#0 -> output:#PWR_LED#13
- U$101, U$407: device output:#SCL#0 -> output:#JP1#14
- U$102, U$408: device output:#STAT#3 -> output:BUZZER14
- U$103: device output:##RST##7 -> output:STAT0
- U$104: device output:##TRIG##6 -> output:PWR0
- U$105: device output:USER12 -> SparkFun-Aesthetics:QWIIC_5MM
- U$106: device output:#PWR_LED#13 -> output:BUZZER1
- U$107: device output:#JP1#14 -> output:#I2C#0
- U$108, U$126: device output:BUZZER14 -> output:#GND#0
- U$109, U$397, U$91: device output:STAT0 -> output:#GND#0
- U$110: device output:PWR0 -> output:#3V3#0
- U$111: device SparkFun-Aesthetics:QWIIC_4MM -> output:#SDA#0
- U$112: device SparkFun-Aesthetics:QWIIC_5MM -> output:#SCL#0
- U$113: device output:BUZZER1 -> output:#STAT#3
- U$114: device output:#I2C#0 -> output:##RST##7
- U$115, U$404, U$98: device output:#GND#0 -> output:##TRIG##6
- U$116, U$133: device output:#GND#0 -> output:USER12
- U$117: device output:#3V3#0 -> output:#PWR_LED#13
- U$118: device output:#SDA#0 -> output:#JP1#14
- U$119: device output:#SCL#0 -> output:BUZZER14
- U$120: device output:#STAT#3 -> output:STAT0
- U$121: device output:##RST##7 -> output:PWR0
- U$122: device output:##TRIG##6 -> SparkFun-Aesthetics:QWIIC_5MM
- U$123: device output:USER12 -> output:BUZZER1
- U$124: device output:#PWR_LED#13 -> output:#I2C#0
- U$125, U$143: device output:#JP1#14 -> output:#GND#0
- U$127: device output:STAT0 -> output:#3V3#0
- U$128: device output:PWR0 -> output:#SDA#0
- U$129: device SparkFun-Aesthetics:QWIIC_4MM -> output:#SCL#0
- U$130: device SparkFun-Aesthetics:QWIIC_5MM -> output:#STAT#3
- U$131: device output:BUZZER1 -> output:##RST##7
- U$132: device output:#I2C#0 -> output:##TRIG##6
- U$134, U$151: device output:#GND#0 -> output:#PWR_LED#13
- U$135: device output:#3V3#0 -> output:#JP1#14
- U$136: device output:#SDA#0 -> output:BUZZER14
- U$137: device output:#SCL#0 -> output:STAT0
- U$138: device output:#STAT#3 -> output:PWR0
- U$139: device output:##RST##7 -> SparkFun-Aesthetics:QWIIC_5MM
- U$14, U$326: device output:PWR0 -> SparkFun-Aesthetics:QWIIC_5MM
- U$140: device output:##TRIG##6 -> output:BUZZER1
- U$141: device output:USER12 -> output:#I2C#0
- U$142, U$160: device output:#PWR_LED#13 -> output:#GND#0
- U$144: device output:BUZZER14 -> output:#3V3#0
- U$145: device output:STAT0 -> output:#SDA#0
- U$146: device output:PWR0 -> output:#SCL#0
- U$147: device SparkFun-Aesthetics:QWIIC_4MM -> output:#STAT#3
- U$148: device SparkFun-Aesthetics:QWIIC_5MM -> output:##RST##7
- U$149: device output:BUZZER1 -> output:##TRIG##6
- U$150: device output:#I2C#0 -> output:USER12
- U$152, U$169: device output:#GND#0 -> output:#JP1#14
- U$153: device output:#3V3#0 -> output:BUZZER14
- U$154: device output:#SDA#0 -> output:STAT0
- U$155: device output:#SCL#0 -> output:PWR0
- U$156: device output:#STAT#3 -> SparkFun-Aesthetics:QWIIC_5MM
- U$157: device output:##RST##7 -> output:BUZZER1
- U$158: device output:##TRIG##6 -> output:#I2C#0
- U$159, U$177: device output:USER12 -> output:#GND#0
- U$161: device output:#JP1#14 -> output:#3V3#0
- U$162: device output:BUZZER14 -> output:#SDA#0
- U$163: device output:STAT0 -> output:#SCL#0
- U$164: device output:PWR0 -> output:#STAT#3
- U$165: device SparkFun-Aesthetics:QWIIC_4MM -> output:##RST##7
- U$166: device SparkFun-Aesthetics:QWIIC_5MM -> output:##TRIG##6
- U$167: device output:BUZZER1 -> output:USER12
- U$168: device output:#I2C#0 -> output:#PWR_LED#13
- U$170, U$187: device output:#GND#0 -> output:BUZZER14
- U$171: device output:#3V3#0 -> output:STAT0
- U$172: device output:#SDA#0 -> output:PWR0
- U$173: device output:#SCL#0 -> SparkFun-Aesthetics:QWIIC_5MM
- U$174: device output:#STAT#3 -> output:BUZZER1
- U$175: device output:##RST##7 -> output:#I2C#0
- U$176, U$194: device output:##TRIG##6 -> output:#GND#0
- U$178: device output:#PWR_LED#13 -> output:#3V3#0
- U$179: device output:#JP1#14 -> output:#SDA#0
- U$180: device output:BUZZER14 -> output:#SCL#0
- U$181: device output:STAT0 -> output:#STAT#3
- U$182: device output:PWR0 -> output:##RST##7
- U$183: device SparkFun-Aesthetics:QWIIC_4MM -> output:##TRIG##6
- U$184: device SparkFun-Aesthetics:QWIIC_5MM -> output:USER12
- U$185: device output:BUZZER1 -> output:#PWR_LED#13
- U$186: device output:#I2C#0 -> output:#JP1#14
- U$188, U$205: device output:#GND#0 -> output:STAT0
- U$189: device output:#3V3#0 -> output:PWR0
- U$190: device output:#SDA#0 -> SparkFun-Aesthetics:QWIIC_5MM
- U$191: device output:#SCL#0 -> output:BUZZER1
- U$192: device output:#STAT#3 -> output:#I2C#0
- U$193, U$211: device output:##RST##7 -> output:#GND#0
- U$195: device output:USER12 -> output:#3V3#0
- U$196: device output:#PWR_LED#13 -> output:#SDA#0
- U$197: device output:#JP1#14 -> output:#SCL#0
- U$198: device output:BUZZER14 -> output:#STAT#3
- U$199: device output:STAT0 -> output:##RST##7
- U$20, U$327: device SparkFun-Aesthetics:QWIIC_4MM -> output:BUZZER1
- U$200: device output:PWR0 -> output:##TRIG##6
- U$201: device SparkFun-Aesthetics:QWIIC_4MM -> output:USER12
- U$202: device SparkFun-Aesthetics:QWIIC_5MM -> output:#PWR_LED#13
- U$203: device output:BUZZER1 -> output:#JP1#14
- U$204: device output:#I2C#0 -> output:BUZZER14
- U$206, U$223: device output:#GND#0 -> output:PWR0
- U$207: device output:#3V3#0 -> SparkFun-Aesthetics:QWIIC_5MM
- U$208: device output:#SDA#0 -> output:BUZZER1
- U$209: device output:#SCL#0 -> output:#I2C#0
- U$21, U$328: device SparkFun-Aesthetics:QWIIC_5MM -> output:#I2C#0
- U$210, U$228: device output:#STAT#3 -> output:#GND#0
- U$212: device output:##TRIG##6 -> output:#3V3#0
- U$213: device output:USER12 -> output:#SDA#0
- U$214: device output:#PWR_LED#13 -> output:#SCL#0
- U$215: device output:#JP1#14 -> output:#STAT#3
- U$216: device output:BUZZER14 -> output:##RST##7
- U$217: device output:STAT0 -> output:##TRIG##6
- U$218: device output:PWR0 -> output:USER12
- U$219: device SparkFun-Aesthetics:QWIIC_4MM -> output:#PWR_LED#13
- U$220: device SparkFun-Aesthetics:QWIIC_5MM -> output:#JP1#14
- U$221: device output:BUZZER1 -> output:BUZZER14
- U$222: device output:#I2C#0 -> output:STAT0
- U$224, U$241: device output:#GND#0 -> SparkFun-Aesthetics:QWIIC_5MM
- U$225: device output:#3V3#0 -> output:BUZZER1
- U$226: device output:#SDA#0 -> output:#I2C#0
- U$227, U$245: device output:#SCL#0 -> output:#GND#0
- U$229: device output:##RST##7 -> output:#3V3#0
- U$23, U$329, U$347, U$41: device output:BUZZER1 -> output:#GND#0
- U$230: device output:##TRIG##6 -> output:#SDA#0
- U$231: device output:USER12 -> output:#SCL#0
- U$232: device output:#PWR_LED#13 -> output:#STAT#3
- U$233: device output:#JP1#14 -> output:##RST##7
- U$234: device output:BUZZER14 -> output:##TRIG##6
- U$235: device output:STAT0 -> output:USER12
- U$236: device output:PWR0 -> output:#PWR_LED#13
- U$237: device SparkFun-Aesthetics:QWIIC_4MM -> output:#JP1#14
- U$238: device SparkFun-Aesthetics:QWIIC_5MM -> output:BUZZER14
- U$239: device output:BUZZER1 -> output:STAT0
- U$24, U$312, U$330: device output:#I2C#0 -> output:#GND#0
- U$240: device output:#I2C#0 -> output:PWR0
- U$242, U$259: device output:#GND#0 -> output:BUZZER1
- U$243: device output:#3V3#0 -> output:#I2C#0
- U$244, U$262: device output:#SDA#0 -> output:#GND#0
- U$246: device output:#STAT#3 -> output:#3V3#0
- U$247: device output:##RST##7 -> output:#SDA#0
- U$248: device output:##TRIG##6 -> output:#SCL#0
- U$249: device output:USER12 -> output:#STAT#3
- U$25, U$314, U$331: device output:#GND#0 -> output:#3V3#0
- U$250: device output:#PWR_LED#13 -> output:##RST##7
- U$251: device output:#JP1#14 -> output:##TRIG##6
- U$252: device output:BUZZER14 -> output:USER12
- U$253: device output:STAT0 -> output:#PWR_LED#13
- U$254: device output:PWR0 -> output:#JP1#14
- U$255: device SparkFun-Aesthetics:QWIIC_4MM -> output:BUZZER14
- U$256: device SparkFun-Aesthetics:QWIIC_5MM -> output:STAT0
- U$257: device output:BUZZER1 -> output:PWR0
- U$258: device output:#I2C#0 -> SparkFun-Aesthetics:QWIIC_5MM
- U$26, U$332, U$349, U$43: device output:#GND#0 -> output:#SDA#0
- U$260, U$277: device output:#GND#0 -> output:#I2C#0
- U$261, U$279: device output:#3V3#0 -> output:#GND#0
- U$263: device output:#SCL#0 -> output:#3V3#0
- U$264: device output:#STAT#3 -> output:#SDA#0
- U$265: device output:##RST##7 -> output:#SCL#0
- U$266: device output:##TRIG##6 -> output:#STAT#3
- U$267: device output:USER12 -> output:##RST##7
- U$268: device output:#PWR_LED#13 -> output:##TRIG##6
- U$269: device output:#JP1#14 -> output:USER12
- U$27, U$333: device output:#3V3#0 -> output:#SCL#0
- U$270: device output:BUZZER14 -> output:#PWR_LED#13
- U$271: device output:STAT0 -> output:#JP1#14
- U$272: device output:PWR0 -> output:BUZZER14
- U$273, U$3: device SparkFun-Aesthetics:QWIIC_4MM -> output:STAT0
- U$274: device SparkFun-Aesthetics:QWIIC_5MM -> output:PWR0
- U$275: device output:BUZZER1 -> SparkFun-Aesthetics:QWIIC_5MM
- U$276: device output:#I2C#0 -> output:BUZZER1
- U$28, U$334: device output:#SDA#0 -> output:#STAT#3
- U$280: device output:#SDA#0 -> output:#3V3#0
- U$281: device output:#SCL#0 -> output:#SDA#0
- U$282: device output:#STAT#3 -> output:#SCL#0
- U$283: device output:##RST##7 -> output:#STAT#3
- U$284: device output:##TRIG##6 -> output:##RST##7
- U$285: device output:USER12 -> output:##TRIG##6
- U$286: device output:#PWR_LED#13 -> output:USER12
- U$287: device output:#JP1#14 -> output:#PWR_LED#13
- U$288: device output:BUZZER14 -> output:#JP1#14
- U$289: device output:STAT0 -> output:BUZZER14
- U$29, U$335: device output:#SCL#0 -> output:##RST##7
- U$290: device output:PWR0 -> output:STAT0
- U$291: device SparkFun-Aesthetics:QWIIC_4MM -> output:PWR0
- U$30, U$336: device output:#STAT#3 -> output:##TRIG##6
- U$309: device SparkFun-Aesthetics:QWIIC_4MM -> SparkFun-Aesthetics:QWIIC_5MM
- U$31, U$337: device output:##RST##7 -> output:USER12
- U$310: device SparkFun-Aesthetics:QWIIC_5MM -> output:BUZZER1
- U$311: device output:BUZZER1 -> output:#I2C#0
- U$315: device output:#3V3#0 -> output:#SDA#0
- U$316: device output:#SDA#0 -> output:#SCL#0
- U$317: device output:#SCL#0 -> output:#STAT#3
- U$318: device output:#STAT#3 -> output:##RST##7
- U$319: device output:##RST##7 -> output:##TRIG##6
- U$32, U$338: device output:##TRIG##6 -> output:#PWR_LED#13
- U$320: device output:##TRIG##6 -> output:USER12
- U$321: device output:USER12 -> output:#PWR_LED#13
- U$322: device output:#PWR_LED#13 -> output:#JP1#14
- U$323: device output:#JP1#14 -> output:BUZZER14
- U$324: device output:BUZZER14 -> output:STAT0
- U$325, U$4: device output:STAT0 -> output:PWR0
- U$33, U$339: device output:USER12 -> output:#JP1#14
- U$34, U$340: device output:#PWR_LED#13 -> output:BUZZER14
- U$341, U$35: device output:#JP1#14 -> output:STAT0
- U$342, U$36: device output:BUZZER14 -> output:PWR0
- U$343, U$37: device output:STAT0 -> SparkFun-Aesthetics:QWIIC_5MM
- U$344, U$38: device output:PWR0 -> output:BUZZER1
- U$345, U$39: device SparkFun-Aesthetics:QWIIC_4MM -> output:#I2C#0
- U$346, U$364, U$40, U$58: device SparkFun-Aesthetics:QWIIC_5MM -> output:#GND#0
- U$348, U$42: device output:#I2C#0 -> output:#3V3#0
- U$350, U$367, U$44, U$61: device output:#GND#0 -> output:#SCL#0
- U$351, U$45: device output:#3V3#0 -> output:#STAT#3
- U$352, U$46: device output:#SDA#0 -> output:##RST##7
- U$353, U$47: device output:#SCL#0 -> output:##TRIG##6
- U$354, U$48: device output:#STAT#3 -> output:USER12
- U$355, U$49: device output:##RST##7 -> output:#PWR_LED#13
- U$356, U$50: device output:##TRIG##6 -> output:#JP1#14
- U$357, U$51: device output:USER12 -> output:BUZZER14
- U$358, U$52: device output:#PWR_LED#13 -> output:STAT0
- U$359, U$53: device output:#JP1#14 -> output:PWR0
- U$360, U$54: device output:BUZZER14 -> SparkFun-Aesthetics:QWIIC_5MM
- U$361, U$55: device output:STAT0 -> output:BUZZER1
- U$362, U$56: device output:PWR0 -> output:#I2C#0
- U$363, U$381, U$57, U$75: device SparkFun-Aesthetics:QWIIC_4MM -> output:#GND#0
- U$365, U$59: device output:BUZZER1 -> output:#3V3#0
- U$366, U$60: device output:#I2C#0 -> output:#SDA#0
- U$368, U$385, U$62, U$79: device output:#GND#0 -> output:#STAT#3
- U$369, U$63: device output:#3V3#0 -> output:##RST##7
- U$370, U$64: device output:#SDA#0 -> output:##TRIG##6
- U$371, U$65: device output:#SCL#0 -> output:USER12
- U$372, U$66: device output:#STAT#3 -> output:#PWR_LED#13
- U$373, U$67: device output:##RST##7 -> output:#JP1#14
- U$374, U$68: device output:##TRIG##6 -> output:BUZZER14
- U$375, U$69: device output:USER12 -> output:STAT0
- U$376, U$70: device output:#PWR_LED#13 -> output:PWR0
- U$377, U$71: device output:#JP1#14 -> SparkFun-Aesthetics:QWIIC_5MM
- U$378, U$72: device output:BUZZER14 -> output:BUZZER1
- U$379, U$73: device output:STAT0 -> output:#I2C#0
- U$380, U$398, U$74, U$92: device output:PWR0 -> output:#GND#0
- U$382, U$76: device SparkFun-Aesthetics:QWIIC_5MM -> output:#3V3#0
- U$383, U$77: device output:BUZZER1 -> output:#SDA#0
- U$384, U$78: device output:#I2C#0 -> output:#SCL#0
- U$386, U$403, U$80, U$97: device output:#GND#0 -> output:##RST##7
- U$387, U$81: device output:#3V3#0 -> output:##TRIG##6
- U$388, U$82: device output:#SDA#0 -> output:USER12
- U$389, U$83: device output:#SCL#0 -> output:#PWR_LED#13
- U$390, U$84: device output:#STAT#3 -> output:#JP1#14
- U$391, U$85: device output:##RST##7 -> output:BUZZER14
- U$392, U$86: device output:##TRIG##6 -> output:STAT0
- U$393, U$87: device output:USER12 -> output:PWR0
- U$394, U$88: device output:#PWR_LED#13 -> SparkFun-Aesthetics:QWIIC_5MM
- U$395, U$89: device output:#JP1#14 -> output:BUZZER1
- U$396, U$90: device output:BUZZER14 -> output:#I2C#0
- U$399, U$93: device SparkFun-Aesthetics:QWIIC_4MM -> output:#3V3#0
- U$400, U$94: device SparkFun-Aesthetics:QWIIC_5MM -> output:#SDA#0
- U$401, U$95: device output:BUZZER1 -> output:#SCL#0
- U$402, U$96: device output:#I2C#0 -> output:#STAT#3
- U$405, U$99: device output:#3V3#0 -> output:USER12
- moved U$321 148.1 mm to (2.84, 89.9), turned to 90 degrees
- moved U$215 145.7 mm to (5.61, 68.2), turned to 90 degrees
- moved U$317 145.7 mm to (5.61, 94.1)
- moved U$312 144.6 mm to (8.86, 81.7)
- moved LOGO21 140.6 mm to (149.7, 5.99)
- moved U$309 139.9 mm to (13.1, 88.0), flipped to the bottom
- moved U$216 139.0 mm to (8.89, 73.5), turned to 90 degrees
- moved U$205 138.5 mm to (6.03, 70.5), flipped to the top
- moved U$206 138.0 mm to (6.03, 59.0), flipped to the top
- moved U$105 137.7 mm to (13.1, 36.2)
- moved U$323 137.4 mm to (12.8, 86.5)
- moved U$213 136.2 mm to (14.0, 55.8), turned to 90 degrees
- moved U$104 135.4 mm to (6.03, 33.1), flipped to the top
- moved U$108 135.2 mm to (8.86, 29.9), turned to 90 degrees
- moved U$103 134.4 mm to (6.03, 44.6), flipped to the top
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- renumbered U$417 to LOGO96
